File: KiCad/transciever.kicad_sch (KiCad schematic)
At the start: 4 parts, among them J2 Conn_01x03, U4 MCP2551-I-SN

Commit message: errors cadlab
Connections:
- net BUS_CANH: no longer names the net of J2.1 (Pin_1), R13.1, U4.7 (CANH)
- net BUS_CANL: no longer names the net of J2.2 (Pin_2), R13.2, U4.6 (CANL)
Changed lines of the file:
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@@
-	(wire
-		(pts
-			(xy 154.94 92.71) (xy 154.94 96.52)
-		)
-		(stroke
-			(width 0)
-			(type default)
-		)
-	)
 	(wire
 		(pts
@@
 	(wire
 		(pts
-			(xy 154.94 114.3) (xy 154.94 104.14)
-		)
-		(stroke
-			(width 0)
-			(type default)
-		)
-	)
-	(wire
-		(pts
 			(xy 162.56 99.06) (xy 162.56 96.52)
 		)
@@
 	(wire
 		(pts
-			(xy 158.75 114.3) (xy 154.94 114.3)
-		)
-		(stroke
-			(width 0)
-			(type default)
-		)
-	)
-	(wire
-		(pts
 			(xy 123.19 97.79) (xy 124.46 97.79)
 		)
@@
 		(pts
 			(xy 123.19 102.87) (xy 124.46 102.87)
-		)
-		(stroke
-			(width 0)
-			(type default)
-		)
-	)
-	(wire
-		(pts
-			(xy 158.75 92.71) (xy 154.94 92.71)
 		)
 		(stroke
@@
 				(hide yes)
 			)
-		)
-	)
-	(global_label "BUS_CANL"
-		(shape input)
-		(at 158.75 114.3 0)
-		(fields_autoplaced yes)
-		(effects
-			(font
-				(size 1.27 1.27)
-			)
-			(justify left)
-		)
-		(property "Intersheetrefs" "${INTERSHEET_REFS}"
-			(at 171.23 114.3 0)
-			(effects
-				(font
-					(size 1.27 1.27)
-				)
-				(justify left)
-				(hide yes)
-			)
-		)
-	)
-	(global_label "BUS_CANH"
-		(shape input)
-		(at 158.75 92.71 0)
-		(fields_autoplaced yes)
-		(effects
-			(font
-				(size 1.27 1.27)
-			)
-			(justify left)
-		)
-		(property "Intersheetrefs" "${INTERSHEET_REFS}"
-			(at 171.5324 92.71 0)
-			(effects
-				(font
-					(size 1.27 1.27)
-				)
-				(justify left)
-				(hide yes)
-			)
