File: KiCad/transciever.kicad_sch (KiCad schematic)
At the start: 4 parts, among them J2 Conn_01x03, U4 MCP2551-I-SN

Commit message: errors pcb
Parts:
- removed J2: Conn_01x03, Connector_PinHeader_2.54mm:PinHeader_1x03_P2.54mm_Vertical, symbol Connector_Generic:Conn_01x03
- added J5: DE9_Pins, Connector_Dsub:DSUB-9_Pins_Vertical_P2.77x2.84mm, symbol Connector:DE9_Pins
- added R15: 10k, Resistor_SMD:R_0805_2012Metric_Pad1.20x1.40mm_HandSolder, symbol Device:R
Connections:
- net GND: now also J5.1, R15.2; no longer U4.8 (Rs)
- net CANH: now reaches R13.1, U4.7 (CANH)
- net CANH: now also J5.3
- net CANL: now reaches R13.2, U4.6 (CANL)
- net CANL: now also J5.7
- new net Rs: R15.1, U4.8 (Rs)
- new net UART_RX: J5.9
- new net UART_TX: J5.5
- no-connect marks 1 -> 5
