File: KiCad/sensor_llum.kicad_sch (KiCad schematic)
At the start: 0 parts

Commit message: he canviat el micro
Parts:
- added BH1750: ~, symbol PROJECTE_LLUMS:BH1750
- added C1: 100nF, symbol Device:C
- added R14, R15: 4.7K, symbol Device:R
Connections:
- new net 3V3: BH1750.1 (VCC), C1.1, R14.1, R15.1
- new net GND: BH1750.2 (ADDR), BH1750.3 (GND), C1.2
- new net I2C_SCL: BH1750.6 (SCL), R15.2
- new net I2C_SDA: BH1750.4 (SDA), R14.2
Other:
- note added: "Pull up a prop de VCC del sensor"
- note added: "SENSOR LLUM"

Commit message: ERC i footprints
Parts:
- removed BH1750: ~, symbol PROJECTE_LLUMS:BH1750
- removed C1: 100nF, symbol Device:C
- removed R14, R15: 4.7K, symbol Device:R
- added C9: 100nF, Capacitor_SMD:C_0805_2012Metric_Pad1.18x1.45mm_HandSolder, symbol Device:C
- added R19, R20: 4.7k, Resistor_SMD:R_0805_2012Metric_Pad1.20x1.40mm_HandSolder, symbol Device:R
- added U1: BH1750FVI-TR, BH1750FVI-TR:XDCR_BH1750FVI-TR, symbol BH1750FVI-TR:BH1750FVI-TR
Connections:
- net 3V3: now also C9.1, R19.1, R20.1, U1.1 (VCC)
- net GND: now also C9.2, U1.2 (ADDR), U1.3 (GND)
- net I2C_SCL: now also R19.2, U1.6 (SCL)
- net I2C_SDA: now also R20.2, U1.4 (SDA)
- no-connect marks 0 -> 1

Commit message: placement (falten LEDs)
Parts:
- U1: footprint BH1750FVI-TR:XDCR_BH1750FVI-TR -> footprints:XDCR_BH1750FVI-TR
Changed lines of the file:
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@@
 			)
 		)
-		(property "Footprint" "BH1750FVI-TR:XDCR_BH1750FVI-TR"
+		(property "Footprint" "footprints:XDCR_BH1750FVI-TR"
 			(at 151.13 95.25 0)
 			(effects

Commit message: errors cadlab
Parts:
- removed R20: 4.7k, Resistor_SMD:R_0805_2012Metric_Pad1.20x1.40mm_HandSolder, symbol Device:R
- added R14: 4.7k, Resistor_SMD:R_0805_2012Metric_Pad1.20x1.40mm_HandSolder, symbol Device:R
Connections:
- net 3V3: now also R19.2, R14.2; no longer R19.1
- net I2C_SCL: no longer names the net of U1.6 (SCL)
- net I2C_SCL: now also R19.1; no longer R19.2
- net I2C_SDA: no longer names the net of U1.4 (SDA)
- net I2C_SDA: now also R14.1
Other:
- moved on the sheet: R19

Commit message: errors pcb
Connections:
- net SDA: now reaches R14.1, U1.4 (SDA)
- net SCL: now reaches R19.1, U1.6 (SCL)
Changed lines of the file:
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@@
+		)
+	)
+	(label "SCL"
+		(at 132.08 95.25 0)
+		(effects
+			(font
+				(size 1.27 1.27)
+			)
+			(justify left bottom)
+		)
+	)
+	(label "SDA"
+		(at 125.73 97.79 0)
+		(effects
+			(font
+				(size 1.27 1.27)
+			)
+			(justify left bottom)
 		)
 	)
