File: KiCad/microcontrolador.kicad_sch (KiCad schematic)
At the start: 17 parts, among them J2 DE9_Pins_MountingHoles, J3 Conn_01x05, J5 DE9_Pins_MountingHoles, U4 MCP2551-I-SN, U7 PIC24HJ128GP502, Y1 8MHz

Commit message: algo de routing
Parts:
- added TP_SCL1, TP_SDA1: TestPoint, Connector_PinHeader_2.54mm:PinHeader_1x01_P2.54mm_Vertical, symbol Connector:TestPoint
Connections:
- net 5V is gone; now on net +5V: J3.2 (Pin_2)
- net I2C_SCL: now also TP_SCL1.1
- net I2C_SDA: now also TP_SDA1.1
Changed lines of the file:
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@@
+	)
+	(junction
+		(at 142.24 90.17)
+		(diameter 0)
+		(color 0 0 0 0)
 	)
 	(junction
@@
 		(color 0 0 0 0)
 	)
+	(junction
+		(at 146.05 92.71)
+		(diameter 0)
+		(color 0 0 0 0)
+	)
 	(no_connect
 		(at 236.22 113.03)
@@
 	(wire
 		(pts
+			(xy 146.05 92.71) (xy 147.32 92.71)
+		)
+		(stroke
+			(width 0)
+			(type default)
+		)
+	)
+	(wire
+		(pts
 			(xy 232.41 110.49) (xy 232.41 111.76)
 		)
@@
 	(wire
 		(pts
+			(xy 128.27 92.71) (xy 146.05 92.71)
+		)
+		(stroke
+			(width 0)
+			(type default)
+		)
+	)
+	(wire
+		(pts
 			(xy 215.9 128.27) (xy 219.71 128.27)
 		)
@@
 	(wire
 		(pts
-			(xy 130.81 92.71) (xy 128.27 92.71)
-		)
-		(stroke
-			(width 0)
-			(type default)
-		)
-	)
-	(wire
-		(pts
 			(xy 130.81 85.09) (xy 128.27 85.09)
 		)
@@
 	(wire
 		(pts
+			(xy 128.27 90.17) (xy 142.24 90.17)
+		)
+		(stroke
+			(width 0)
+			(type default)
+		)
+	)
+	(wire
+		(pts
 			(xy 71.12 118.11) (xy 71.12 114.3)
 		)
@@
 	(wire
 		(pts
-			(xy 130.81 90.17) (xy 128.27 90.17)
+			(xy 143.51 90.17) (xy 142.24 90.17)
 		)
 		(stroke
@@
 	(global_label "I2C_SDA"
 		(shape input)
-		(at 130.81 92.71 0)
+		(at 147.32 92.71 0)
 		(fields_autoplaced yes)
 		(effects
@@
 		)
 		(property "Intersheetrefs" "${INTERSHEET_REFS}"
-			(at 141.4152 92.71 0)
+			(at 157.9252 92.71 0)
 			(effects
 				(font
@@
 	(global_label "I2C_SCL"
 		(shape input)
-		(at 130.81 90.17 0)
+		(at 143.51 90.17 0)
 		(fields_autoplaced yes)
 		(effects
@@
 		)
 		(property "Intersheetrefs" "${INTERSHEET_REFS}"
-			(at 141.3547 90.17 0)
+			(at 154.0547 90.17 0)
 			(effects
 				(font
@@
 	)
 	(symbol
+		(lib_id "Connector:TestPoint")
+		(at 142.24 90.17 0)
+		(unit 1)
+		(exclude_from_sim no)
+		(in_bom yes)
+		(on_board yes)
+		(dnp no)
+		(property "Reference" "TP_SCL1"
+			(at 144.78 84.328 0)
+			(effects
+				(font
+					(size 1.27 1.27)
+				)
+				(justify left)
+			)
+		)
+		(property "Value" "TestPoint"
+			(at 144.78 86.868 0)
+			(effects
+				(font
+					(size 1.27 1.27)
+				)
+				(justify left)
+			)
+		)
+		(property "Footprint" "Connector_PinHeader_2.54mm:PinHeader_1x01_P2.54mm_Vertical"
+			(at 147.32 90.17 0)
+			(effects
+				(font
+					(size 1.27 1.27)
+				)
+				(hide yes)
+			)
+		)
+		(property "Datasheet" "~"
+			(at 147.32 90.17 0)
+			(effects
+				(font
+					(size 1.27 1.27)
+				)
+				(hide yes)
+			)
+		)
+		(property "Description" "test point"
+			(at 142.24 90.17 0)
+			(effects
+				(font
+					(size 1.27 1.27)
+				)
+				(hide yes)
+			)
+		)
+		(pin "1"
+		)
+		(instances
+			(project ""
+				(path "/b4874c87-978f-427f-bc45-3635f8629977/65403977-6a27-47ce-ace7-4876548c1d8f"
+					(reference "TP_SCL1")
+					(unit 1)
+				)
+			)
+		)
+	)
+	(symbol
 		(lib_id "Device:R")
 		(at 55.88 106.68 180)
@@
 				(path "/b4874c87-978f-427f-bc45-3635f8629977/65403977-6a27-47ce-ace7-4876548c1d8f"
 					(reference "R1")
+					(unit 1)
+				)
+			)
+		)
+	)
+	(symbol
+		(lib_id "Connector:TestPoint")
+		(at 146.05 92.71 0)
+		(mirror x)
+		(unit 1)
+		(exclude_from_sim no)
+		(in_bom yes)
+		(on_board yes)
+		(dnp no)
+		(property "Reference" "TP_SDA1"
+			(at 148.59 98.552 0)
+			(effects
+				(font
+					(size 1.27 1.27)
+				)
+				(justify left)
+			)
+		)
+		(property "Value" "TestPoint"
+			(at 148.59 96.012 0)
+			(effects
+				(font
+					(size 1.27 1.27)
+				)
+				(justify left)
+			)
+		)
+		(property "Footprint" "Connector_PinHeader_2.54mm:PinHeader_1x01_P2.54mm_Vertical"
+			(at 151.13 92.71 0)
+			(effects
+				(font
+					(size 1.27 1.27)
+				)
+				(hide yes)
+			)
+		)
+		(property "Datasheet" "~"
+			(at 151.13 92.71 0)
+			(effects
+				(font
+					(size 1.27 1.27)
+				)
+				(hide yes)
+			)
+		)
+		(property "Description" "test point"
+			(at 146.05 92.71 0)
+			(effects
+				(font
+					(size 1.27 1.27)
+				)
+				(hide yes)
+			)
+		)
+		(pin "1"
+		)
+		(instances
+			(project "PROJECTE_LLUMS"
+				(path "/b4874c87-978f-427f-bc45-3635f8629977/65403977-6a27-47ce-ace7-4876548c1d8f"
+					(reference "TP_SDA1")
 					(unit 1)
 				)
@@
 			)
 		)
-		(property "Value" "5V"
+		(property "Value" "+5V"
 			(at 90.17 154.94 0)
 			(effects

Commit message: coses
Parts:
- added R50: 0, Resistor_SMD:R_0805_2012Metric_Pad1.20x1.40mm_HandSolder, symbol Device:R
Connections:
- net GND: now also R50.2
- new net GNDPWR: R50.1
Changed lines of the file:
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@@
+	(wire
+		(pts
+			(xy 154.94 33.02) (xy 154.94 36.83)
+		)
+		(stroke
+			(width 0)
+			(type default)
+		)
+	)
 	(wire
 		(pts
@@
 	(wire
 		(pts
+			(xy 168.91 33.02) (xy 165.1 33.02)
+		)
+		(stroke
+			(width 0)
+			(type default)
+		)
+	)
+	(wire
+		(pts
 			(xy 215.9 127) (xy 214.63 127)
 		)
@@
 		(pts
 			(xy 215.9 120.65) (xy 219.71 120.65)
+		)
+		(stroke
+			(width 0)
+			(type default)
+		)
+	)
+	(wire
+		(pts
+			(xy 157.48 33.02) (xy 154.94 33.02)
+		)
+		(stroke
+			(width 0)
+			(type default)
+		)
+	)
+	(wire
+		(pts
+			(xy 168.91 38.1) (xy 168.91 33.02)
 		)
 		(stroke
@@
 				(path "/b4874c87-978f-427f-bc45-3635f8629977/65403977-6a27-47ce-ace7-4876548c1d8f"
 					(reference "#PWR018")
+					(unit 1)
+				)
+			)
+		)
+	)
+	(symbol
+		(lib_id "power:GNDPWR")
+		(at 168.91 38.1 0)
+		(unit 1)
+		(exclude_from_sim no)
+		(in_bom yes)
+		(on_board yes)
+		(dnp no)
+		(fields_autoplaced yes)
+		(property "Reference" "#PWR056"
+			(at 168.91 43.18 0)
+			(effects
+				(font
+					(size 1.27 1.27)
+				)
+				(hide yes)
+			)
+		)
+		(property "Value" "GNDPWR"
+			(at 168.783 41.91 0)
+			(effects
+				(font
+					(size 1.27 1.27)
+				)
+			)
+		)
+		(property "Footprint" ""
+			(at 168.91 39.37 0)
+			(effects
+				(font
+					(size 1.27 1.27)
+				)
+				(hide yes)
+			)
+		)
+		(property "Datasheet" ""
+			(at 168.91 39.37 0)
+			(effects
+				(font
+					(size 1.27 1.27)
+				)
+				(hide yes)
+			)
+		)
+		(property "Description" "Power symbol creates a global label with name \"GNDPWR\" , global ground"
+			(at 168.91 38.1 0)
+			(effects
+				(font
+					(size 1.27 1.27)
+				)
+				(hide yes)
+			)
+		)
+		(pin "1"
+		)
+		(instances
+			(project ""
+				(path "/b4874c87-978f-427f-bc45-3635f8629977/65403977-6a27-47ce-ace7-4876548c1d8f"
+					(reference "#PWR056")
 					(unit 1)
 				)
@@
 	)
 	(symbol
+		(lib_id "power:GND")
+		(at 154.94 36.83 0)
+		(unit 1)
+		(exclude_from_sim no)
+		(in_bom yes)
+		(on_board yes)
+		(dnp no)
+		(fields_autoplaced yes)
+		(property "Reference" "#PWR055"
+			(at 154.94 43.18 0)
+			(effects
+				(font
+					(size 1.27 1.27)
+				)
+				(hide yes)
+			)
+		)
+		(property "Value" "GND"
+			(at 154.94 41.91 0)
+			(effects
+				(font
+					(size 1.27 1.27)
+				)
+			)
+		)
+		(property "Footprint" ""
+			(at 154.94 36.83 0)
+			(effects
+				(font
+					(size 1.27 1.27)
+				)
+				(hide yes)
+			)
+		)
+		(property "Datasheet" ""
+			(at 154.94 36.83 0)
+			(effects
+				(font
+					(size 1.27 1.27)
+				)
+				(hide yes)
+			)
+		)
+		(property "Description" "Power symbol creates a global label with name \"GND\" , ground"
+			(at 154.94 36.83 0)
+			(effects
+				(font
+					(size 1.27 1.27)
+				)
+				(hide yes)
+			)
+		)
+		(pin "1"
+		)
+		(instances
+			(project ""
+				(path "/b4874c87-978f-427f-bc45-3635f8629977/65403977-6a27-47ce-ace7-4876548c1d8f"
+					(reference "#PWR055")
+					(unit 1)
+				)
+			)
+		)
+	)
+	(symbol
 		(lib_id "Connector:TestPoint")
 		(at 142.24 90.17 0)
@@
 					(unit 1)
 				)
+			)
+		)
+	)
+	(symbol
+		(lib_id "Device:R")
+		(at 161.29 33.02 270)
+		(unit 1)
+		(exclude_from_sim no)
+		(in_bom yes)
+		(on_board yes)
+		(dnp no)
+		(property "Reference" "R50"
+			(at 160.274 36.068 0)
+			(effects
+				(font
+					(size 1.27 1.27)
+				)
+			)
+		)
+		(property "Value" "0"
+			(at 162.56 36.83 0)
+			(effects
+				(font
+					(size 1.27 1.27)
+				)
+			)
+		)
+		(property "Footprint" "Resistor_SMD:R_0805_2012Metric_Pad1.20x1.40mm_HandSolder"
+			(at 161.29 31.242 90)
+			(effects
+				(font
+					(size 1.27 1.27)
+				)
+				(hide yes)
+			)
+		)
+		(property "Datasheet" "~"
+			(at 161.29 33.02 0)
+			(effects
+				(font
+					(size 1.27 1.27)
+				)
+				(hide yes)
+			)
+		)
+		(property "Description" "Resistor"
+			(at 161.29 33.02 0)
+			(effects
+				(font
+					(size 1.27 1.27)
+				)
+				(hide yes)
+			)
+		)
+		(pin "1"
+		)
+		(pin "2"
+		)
+		(instances
+			(project "PROJECTE_LLUMS"
+				(path "/b4874c87-978f-427f-bc45-3635f8629977/65403977-6a27-47ce-ace7-4876548c1d8f"
+					(reference "R50")
+					(unit 1)
+				)

Commit message: correccions manel
Connections:
- net +3V3: now also C6.1, C7.1, U7.13 (VDD), U7.28 (AVDD)
- net +5V: no longer C6.1, C7.1, U7.13 (VDD), U7.28 (AVDD)
Changed lines of the file:
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@@
 			)
 		)
-		(property "Value" "+5V"
+		(property "Value" "+3V3"
 			(at 101.6 45.212 0)
 			(effects

Commit message: test points schematic
Parts:
- added D2: LED, LED_SMD:LED_0805_2012Metric_Pad1.15x1.40mm_HandSolder, symbol Device:LED
- added R3: 680, Resistor_SMD:R_0805_2012Metric_Pad1.20x1.40mm_HandSolder, symbol Device:R
- added TP_CANRX1, TP_CANTX1, TP_UART_RX1, TP_UART_TX1: TestPoint, Connector_PinHeader_2.54mm:PinHeader_1x01_P2.54mm_Vertical, symbol Connector:TestPoint
Connections:
- net +3V3: now also R3.1
- net CANRX: now also TP_CANRX1.1
- net CANTX: now also TP_CANTX1.1
- net GND: now also D2.1 (K)
- net UART_RX: now also TP_UART_RX1.1
- net UART_TX: now also TP_UART_TX1.1
- new net: D2.2 (A), R3.2

Commit message: errors CADLAB
Connections:
- net OSC1: now also C2.1, Y1.2; no longer C1.1, Y1.1
- net OSC2: now also C1.1, Y1.1; no longer C2.1, Y1.2
Changed lines of the file:
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@@
 	(wire
 		(pts
-			(xy 77.47 76.2) (xy 90.17 76.2)
+			(xy 77.47 73.66) (xy 90.17 73.66)
 		)
 		(stroke
@@
 	(wire
 		(pts
-			(xy 77.47 80.01) (xy 77.47 76.2)
+			(xy 77.47 80.01) (xy 77.47 73.66)
 		)
 		(stroke
@@
 	(wire
 		(pts
-			(xy 64.77 73.66) (xy 90.17 73.66)
+			(xy 64.77 76.2) (xy 90.17 76.2)
 		)
 		(stroke
@@
 	(wire
 		(pts
-			(xy 64.77 73.66) (xy 64.77 80.01)
+			(xy 64.77 76.2) (xy 64.77 80.01)
 		)
 		(stroke
@@
 		)
 	)
-	(label "OSC1"
-		(at 83.82 73.66 0)
+	(label "OSC2"
+		(at 83.82 76.2 0)
 		(effects
 			(font
@@
 		)
 	)
-	(label "OSC2"
-		(at 83.82 76.2 0)
+	(label "OSC1"
+		(at 83.82 73.66 0)
 		(effects
 			(font

Commit message: push final (?)
Other:
- moved on the sheet: C1, C2, C5, C6, C7, C8, C_out3, D2, J2, J3, J5, R1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
